File: design/Memory.kicad_sch (KiCad schematic)
At the start: 10 parts, among them U14 SST39SF040, U15 SST39SF040, U16 AS6C4008-55PCN, U17 AS6C4008-55PCN

Commit message: Sort out R and C types
Connections:
- net GND: now also U14.16 (GND), U15.16 (GND), U16.16 (VSS), U17.16 (VSS)
- net VCC: now also U14.32 (VCC), U15.32 (VCC), U16.32 (VCC), U17.32 (VCC)

Commit message: Further improvements on CPLD pin placement to improve routing
Parts:
- JP1: footprint (none) -> Connector_PinHeader_2.54mm:PinHeader_1x02_P2.54mm_Vertical
- U14, U15: footprint Package_DIP:DIP-32_W15.24mm_LongPads -> Package_LCC:PLCC-32_THT-Socket
Changed lines of the file:
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@@
 			)
 		)
-		(property "Footprint" "Package_DIP:DIP-32_W15.24mm_LongPads"
+		(property "Footprint" "Package_LCC:PLCC-32_THT-Socket"
 			(at 55.88 95.25 0)
 			(hide yes)
@@
 			)
 		)
-		(property "Footprint" "Package_DIP:DIP-32_W15.24mm_LongPads"
+		(property "Footprint" "Package_LCC:PLCC-32_THT-Socket"
 			(at 107.95 95.25 0)
 			(hide yes)
@@
 			)
 		)
-		(property "Footprint" ""
+		(property "Footprint" "Connector_PinHeader_2.54mm:PinHeader_1x02_P2.54mm_Vertical"
 			(at 67.31 166.37 0)
 			(hide yes)
