File: design/USB.kicad_sch (KiCad schematic)
At the start: 24 parts, among them J4 Backup serial, J5 USB2.0_TypeC, J8 SD Card, SW1 Reset, U1 MCP2221A, U11 UM809SS, U9 USBLC6-2SC6

Commit message: Sort out R and C types
Parts:
- removed R21, R35: 4K7, symbol Device:R
- added R32, R33: 4K7, Resistor_SMD:R_0805_2012Metric_Pad1.20x1.40mm_HandSolder, symbol Device:R
- J5: footprint Connector_USB:USB_C_Receptacle_GCT_USB4135-GF-A_Vertical -> Connector_USB:USB_C_Receptacle_GCT_USB4105-xx-A_16P_TopMnt_Horizontal
- R34: footprint (none) -> Resistor_SMD:R_0805_2012Metric_Pad1.20x1.40mm_HandSolder; LCSC (none) -> C17515; Mouser (none) -> ERJ-6ENF4701V
Connections:
- net GND: now also R34.2
- net USB_N: no longer J5.A6 (D+), J5.B6 (D+), U1.13 (D+), U9.3 (I/O2), U9.4 (I/O2)
- net VCC: now also R33.1
- net at LED10.2 (A): now also R33.2
- net at J4.2 (Pin_2): now also R34.1
- net at LED9.2 (A): now also R32.2; no longer R34.2
- net RESET renamed HWRST
- net HWRST: now also R32.1; no longer R34.1
- new net USB_P: J5.A6 (D+), J5.B6 (D+), U1.13 (D+), U9.3 (I/O2), U9.4 (I/O2)

Commit message: Clean ERCC on schmatic
Parts:
- added J1: SPI CS2, Connector_PinSocket_2.54mm:PinSocket_1x01_P2.54mm_Vertical, symbol Connector:Conn_01x01_Pin
Connections:
- new net SPICS2: J1.1 (Pin_1)
Changed lines of the file:
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@@
 		)
 	)
+	(global_label "SPICS2"
+		(shape input)
+		(at 220.98 151.13 0)
+		(fields_autoplaced yes)
+		(effects
+			(font
+				(size 1.27 1.27)
+			)
+			(justify left)
+		)
+		(property "Intersheetrefs" "${INTERSHEET_REFS}"
+			(at 230.7385 151.13 0)
+			(hide yes)
+			(show_name yes)
+			(do_not_autoplace no)
+			(effects
+				(font
+					(size 1.27 1.27)
+				)
+				(justify left)
+			)
+		)
+	)
 	(global_label "VBUS"
 		(shape input)
@@
 	)
 	(symbol
-		(lib_id "power:PWR_FLAG")
-		(at 63.5 57.15 0)
+		(lib_id "Connector:Conn_01x01_Pin")
+		(at 215.9 151.13 0)
 		(unit 1)
 		(body_style 1)
@@
 		(dnp no)
 		(fields_autoplaced yes)
-		(property "Reference" "#FLG01"
-			(at 63.5 55.245 0)
-			(hide yes)
+		(property "Reference" "J1"
+			(at 216.535 146.05 0)
 			(show_name no)
 			(do_not_autoplace no)
@@
 			)
 		)
-		(property "Value" "PWR_FLAG"
-			(at 63.5 52.07 0)
+		(property "Value" "SPI CS2"
+			(at 216.535 148.59 0)
 			(show_name no)
 			(do_not_autoplace no)
@@
 			)
 		)
-		(property "Footprint" ""
-			(at 63.5 57.15 0)
+		(property "Footprint" "Connector_PinSocket_2.54mm:PinSocket_1x01_P2.54mm_Vertical"
+			(at 215.9 151.13 0)
 			(hide yes)
 			(show_name no)
@@
 		)
 		(property "Datasheet" ""
-			(at 63.5 57.15 0)
+			(at 215.9 151.13 0)
 			(hide yes)
 			(show_name no)
@@
 			)
 		)
-		(property "Description" "Special symbol for telling ERC where power comes from"
-			(at 63.5 57.15 0)
+		(property "Description" "Generic connector, single row, 01x01, script generated"
+			(at 215.9 151.13 0)
 			(hide yes)
 			(show_name no)
@@
 			(project "Simple010"
 				(path "/4f37455c-e998-4ed3-8493-a94956af64c1/7ca0f162-aafd-4dc7-9196-321f0bde09ff"
-					(reference "#FLG01")
+					(reference "J1")
 					(unit 1)
 				)

Commit message: Further improvements on CPLD pin placement to improve routing
Parts:
- removed J5: USB2.0_TypeC, Connector_USB:USB_C_Receptacle_GCT_USB4105-xx-A_16P_TopMnt_Horizontal, symbol Connector:USB_C_Receptacle
- added H1, H2, H3, H4: MountingHole_Pad, MountingHole:MountingHole_3.2mm_M3_Pad_Via, symbol Mechanical:MountingHole_Pad
- added J3: USB_C_Receptacle_USB2.0_16P, Connector_USB:USB_C_Receptacle_HRO_TYPE-C-31-M-12, symbol Connector:USB_C_Receptacle_USB2.0_16P
- J4: footprint (none) -> Connector_PinHeader_2.54mm:PinHeader_1x06_P2.54mm_Vertical
- J8: footprint (none) -> Connector_PinSocket_2.54mm:PinSocket_1x06_P2.54mm_Vertical
- LED10, LED9: footprint (none) -> LED_SMD:LED_0805_2012Metric_Pad1.15x1.40mm_HandSolder
- SW1: footprint (none) -> Button_Switch_SMD:SW_SPST_SKQG_WithoutStem; LCSC (none) -> C318884; Mouser (none) -> C318884
- U1: footprint (none) -> Package_SO:SOIC-14_3.9x8.7mm_P1.27mm; LCSC C130462 -> C640876; Mouser 579-MCP2221A-I/ST -> 579-MCP2221A-I/SL
Connections:
- net VBUS is gone; now on net VCC: C30.2, U9.6 (I/O1)
- net GND: now also H1.1, H2.1, H3.1, H4.1, J3.A1 (GND), J3.A12 (GND), J3.B1 (GND), J3.B12 (GND); no longer C11.1, R12.1
- net USB_N: now also J3.A7 (D-), J3.B7 (D-)
- net USB_P: now also J3.A6 (D+), J3.B6 (D+)
- net VCC: now also J3.A4 (VBUS), J3.A9 (VBUS), J3.B4 (VBUS), J3.B9 (VBUS)
- net at R16.1: now also J3.B5 (CC2)
- net at R15.1: now also J3.A5 (CC1)
- new net GNDS: C11.1, J3.SH (SHIELD), R12.1
- no-connect marks 17 -> 9
Other:
- note added: "(VBUS)"
- moved on the sheet: C11, R12, U9
