File: design/USB.kicad_sch (KiCad schematic)
At the start: 29 parts, among them J1 SPI CS2, J3 USB_C_Receptacle_USB2.0_16P, J4 Backup serial, J8 SD Card, SW1 Reset, U1 MCP2221A, U11 UM809SS, U9 USBLC6-2SC6

Commit message: Fix USB-C connector: update to Korean Hroparts TYPE-C-31-M-12 (C165948)
Corrects J3 from the erroneous C230736 (Jing Extension) to C165948
(Korean Hroparts TYPE-C-31-M-12). Updates schematic, adds datasheet,
and removes the now-resolved note from the INDEX.

Co-Authored-By: Claude Sonnet 4.6 <noreply@anthropic.com>
Parts:
- J3: LCSC C230736 -> C165948
Changed lines of the file:
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@@
 			)
 		)
-		(property "LCSC" "C230736"
+		(property "LCSC" "C165948"
 			(at 49.53 72.39 0)
 			(hide yes)

Commit message: Fix all R/C part numbers: switch to JLCPCB basic parts, correct footprints
- Replace all non-basic LCSC numbers with JLCPCB basic equivalents (no
  extended part setup fees): Samsung MLCCs for caps, UNI-ROYAL 0805W8F
  series for resistors
- Fix C49 footprint: 1210 → 1206 to match Samsung CL31A476MPHNNNE
- Correct previously wrong LCSC numbers (C17512→C17513, C17515→C17673,
  C135808→C96123) and missing R17 part numbers
- Update all Mouser numbers to match the LCSC manufacturer throughout
- Standardise all resistor footprints to HandSolder pad variant
- Update datasheets/INDEX.md with verified basic part table

Co-Authored-By: Claude Sonnet 4.6 <noreply@anthropic.com>
Parts:
- C11: LCSC C62768 -> C1790; Mouser 603-CC0805JRNPO9BN101 -> 187-CL21C101JBANNNC
- C12: now left out of the parts list
- C28: LCSC C106846 -> C13967; Mouser 603-CC0805KKX7R8BB474 -> 187-CL21B474KBFNNNE
- C29: LCSC C89827 -> C15850; Mouser 603-CC0805KKX5R7BB106 -> 187-CL21A106KAYNNNE
- C49: footprint Capacitor_SMD:C_1210_3225Metric_Pad1.33x2.70mm_HandSolder -> Capacitor_SMD:C_1206_3216Metric_Pad1.33x1.80mm_HandSolder; LCSC C135808 -> C96123; Mouser J32MLB7476MPPDTJ -> 187-CL31A476MPHNNNE
- J3: Mouser 649-10118192-0001LF -> 649-10171746-00021LF
- R12: footprint Resistor_SMD:R_0805_2012Metric -> Resistor_SMD:R_0805_2012Metric_Pad1.20x1.40mm_HandSolder; LCSC C107700 -> C17514; Mouser 603-RC0805FR-071ML -> 0805W8F1004T5E
- R15, R16: footprint Resistor_SMD:R_0805_2012Metric -> Resistor_SMD:R_0805_2012Metric_Pad1.20x1.40mm_HandSolder; LCSC C84375 -> C27834; Mouser 603-RC0805FR-075K1L -> 0805W8F5101T5E
- R17: LCSC (none) -> C17513; Mouser (none) -> 0805W8F1001T5E
- R32, R33, R34: LCSC C17515 -> C17673; Mouser ERJ-6ENF4701V -> 0805W8F4701T5E
Changed lines of the file:
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@@
 			)
 		)
-		(property "Mouser" "603-CC0805KKX7R8BB474"
+		(property "Mouser" "187-CL21B474KBFNNNE"
 			(at 204.47 52.07 0)
 			(hide yes)
@@
 			)
 		)
-		(property "LCSC" "C106846"
+		(property "LCSC" "C13967"
 			(at 204.47 52.07 0)
 			(hide yes)
@@
 		(body_style 1)
 		(exclude_from_sim no)
-		(in_bom yes)
+		(in_bom no)
 		(on_board yes)
 		(in_pos_files yes)
@@
 			)
 		)
-		(property "Footprint" "Resistor_SMD:R_0805_2012Metric"
+		(property "Footprint" "Resistor_SMD:R_0805_2012Metric_Pad1.20x1.40mm_HandSolder"
 			(at 48.26 102.87 0)
 			(hide yes)
@@
 			)
 		)
-		(property "Mouser" "603-RC0805FR-071ML"
+		(property "Mouser" "0805W8F1004T5E   "
 			(at 48.26 102.87 0)
 			(hide yes)
@@
 			)
 		)
-		(property "LCSC" "C107700"
+		(property "LCSC" "C17514"
 			(at 48.26 102.87 0)
 			(hide yes)
@@
 			)
 		)
-		(property "Mouser" "603-CC0805JRNPO9BN101"
+		(property "Mouser" "187-CL21C101JBANNNC"
 			(at 48.26 111.76 0)
 			(hide yes)
@@
 			)
 		)
-		(property "LCSC" "C62768"
+		(property "LCSC" "C1790"
 			(at 48.26 111.76 0)
 			(hide yes)
@@
 			)
 		)
-		(property "LCSC" "C17515"
+		(property "LCSC" "C17673"
 			(at 160.02 78.74 0)
 			(hide yes)
@@
 			)
 		)
-		(property "Mouser" "ERJ-6ENF4701V"
+		(property "Mouser" "0805W8F4701T5E"
 			(at 160.02 78.74 0)
 			(hide yes)
@@
 			)
 		)
-		(property "Mouser" "649-10118192-0001LF"
+		(property "Mouser" "649-10171746-00021LF"
 			(at 49.53 72.39 0)
 			(hide yes)
@@
 			)
 		)
-		(property "Footprint" "Capacitor_SMD:C_1210_3225Metric_Pad1.33x2.70mm_HandSolder"
+		(property "Footprint" "Capacitor_SMD:C_1206_3216Metric_Pad1.33x1.80mm_HandSolder"
 			(at 49.53 34.29 0)
 			(hide yes)
@@
 			)
 		)
-		(property "LCSC" "C135808"
+		(property "LCSC" "C96123"
 			(at 49.53 34.29 90)
 			(hide yes)
@@
 			)
 		)
-		(property "Mouser" "J32MLB7476MPPDTJ"
+		(property "Mouser" "187-CL31A476MPHNNNE"
 			(at 49.53 34.29 90)
 			(hide yes)
@@
 			)
 		)
-		(property "Footprint" "Resistor_SMD:R_0805_2012Metric"
+		(property "Footprint" "Resistor_SMD:R_0805_2012Metric_Pad1.20x1.40mm_HandSolder"
 			(at 77.47 64.77 0)
 			(hide yes)
@@
 			)
 		)
-		(property "Mouser" "603-RC0805FR-075K1L"
+		(property "Mouser" "0805W8F5101T5E "
 			(at 87.63 64.77 0)
 			(hide yes)
@@
 			)
 		)
-		(property "LCSC" "C84375"
+		(property "LCSC" "C27834"
 			(at 87.63 64.77 0)
 			(hide yes)
@@
 			)
 		)
-		(property "LCSC" "C17515"
+		(property "LCSC" "C17673"
 			(at 173.99 63.5 0)
 			(hide yes)
@@
 			)
 		)
-		(property "Mouser" "ERJ-6ENF4701V"
+		(property "Mouser" "0805W8F4701T5E"
 			(at 173.99 63.5 0)
 			(hide yes)
@@
 			)
 		)
-		(property "Mouser" "603-CC0805KKX5R7BB106"
+		(property "Mouser" "187-CL21A106KAYNNNE"
 			(at 68.58 35.56 0)
 			(hide yes)
@@
 			)
 		)
-		(property "LCSC" "C89827"
+		(property "LCSC" "C15850"
 			(at 68.58 35.56 0)
 			(hide yes)
@@
 			)
 		)
-		(property "Mouser" ""
+		(property "Mouser" "0805W8F1001T5E"
 			(at 189.23 67.31 0)
 			(hide yes)
@@
 			)
 		)
-		(property "LCSC" ""
+		(property "LCSC" "C17513"
 			(at 189.23 67.31 0)
 			(hide yes)
@@
 			)
 		)
-		(property "Footprint" "Resistor_SMD:R_0805_2012Metric"
+		(property "Footprint" "Resistor_SMD:R_0805_2012Metric_Pad1.20x1.40mm_HandSolder"
 			(at 87.63 55.88 0)
 			(hide yes)
@@
 			)
 		)
-		(property "Mouser" "603-RC0805FR-075K1L"
+		(property "Mouser" "0805W8F5101T5E "
 			(at 87.63 55.88 0)
 			(hide yes)
@@
 			)
 		)
-		(property "LCSC" "C84375"
+		(property "LCSC" "C27834"
 			(at 87.63 55.88 0)
 			(hide yes)
@@
 			)
 		)
-		(property "LCSC" "C17515"
+		(property "LCSC" "C17673"
 			(at 165.1 137.16 0)
 			(hide yes)
@@
 			)
 		)
-		(property "Mouser" "ERJ-6ENF4701V"
+		(property "Mouser" "0805W8F4701T5E"
 			(at 165.1 137.16 0)
 			(hide yes)

Commit message: Change U11 reset supervisor from UM809SS (2.93V) to LM809M3-4.63/NOPB (4.63V)
4.63V threshold gives proper brownout protection on a 5V supply — the 2.93V
part would not trigger until VCC had fallen well below all IC minimum specs.
LM809M3-4.63/NOPB is pin-compatible (same SOT-23-3 footprint), push-pull
active-low, and a JLCPCB Basic part (C2066444). R17 pull-up unchanged.

Co-Authored-By: Claude Sonnet 4.6 <noreply@anthropic.com>
Parts:
- U11: value UM809SS -> LM809M3-4.63/NOPB
Changed lines of the file:
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@@
 			)
 		)
-		(property "Value" "UM809SS"
+		(property "Value" "LM809M3-4.63/NOPB"
 			(at 120.65 76.1999 0)
 			(show_name no)
@@
 			)
 		)
-		(property "Datasheet" ""
+		(property "Datasheet" "https://www.ti.com/lit/ds/symlink/lm809.pdf"
 			(at 127 74.93 0)
 			(hide yes)

Commit message: Update IC part numbers: SST39SF040, AS6C4008, LM809M3-4.63/NOPB
- SST39SF040 (U14/U15): Mouser 579-SST39SF040-70-4I-NHE (PLCC-32,
  industrial grade); LCSC has no PLCC-32 variant in stock
- AS6C4008-55PCN (U16/U17): fix LCSC C62646→C1350141 (was invalid/404);
  Mouser 913-AS6C4008-55PCN has stock, LCSC currently OOS
- LM809M3-4.63/NOPB (U11): add LCSC C2066444 and Mouser part number
  properties to schematic

Co-Authored-By: Claude Sonnet 4.6 <noreply@anthropic.com>
Parts:
- U11: LCSC (none) -> C2066444; Mouser (none) -> 595-LM809M3-4.63NOPB
Changed lines of the file:
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@@
+			)
+		)
+		(property "LCSC" "C2066444"
+			(at 127 74.93 0)
+			(hide yes)
+			(show_name no)
+			(do_not_autoplace no)
+			(effects
+				(font
+					(size 1.27 1.27)
+				)
+			)
+		)
+		(property "Mouser" "595-LM809M3-4.63NOPB"
+			(at 127 74.93 0)
+			(hide yes)
+			(show_name no)
+			(do_not_autoplace no)
+			(effects
+				(font
+					(size 1.27 1.27)
+				)
 			)
 		)

Commit message: Fix even/odd memory bus wiring and route PCB
- Connect U15 (even ROM) and U17 (even RAM) data pins to D8-D15 instead
  of D0-D7: upper byte was completely unconnected, causing half-garbage
  reads and lost writes on all 16-bit accesses
- Reduce R32/R33 LED resistors from 4.7k to 1k (MCP2221A GPIO is 3.3V,
  4.7k gave only 0.26mA — too dim)
- Initial PCB layout and routing

Co-Authored-By: Claude Sonnet 4.6 <noreply@anthropic.com>
Parts:
- R17: value 1k -> 1K
- R32, R33: value 4K7 -> 1K; LCSC C17673 -> C17513; Mouser 0805W8F4701T5E -> 0805W8F1001T5E
Changed lines of the file:
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@@
 			)
 		)
-		(property "Value" "4K7"
+		(property "Value" "1K"
 			(at 162.56 80.0099 0)
 			(show_name no)
@@
 			)
 		)
-		(property "LCSC" "C17673"
+		(property "LCSC" "C17513"
 			(at 160.02 78.74 0)
 			(hide yes)
@@
 			)
 		)
-		(property "Mouser" "0805W8F4701T5E"
+		(property "Mouser" "0805W8F1001T5E"
 			(at 160.02 78.74 0)
 			(hide yes)
@@
 			)
 		)
-		(property "Value" "4K7"
+		(property "Value" "1K"
 			(at 176.53 64.7699 0)
 			(show_name no)
@@
 			)
 		)
-		(property "LCSC" "C17673"
+		(property "LCSC" "C17513"
 			(at 173.99 63.5 0)
 			(hide yes)
@@
 			)
 		)
-		(property "Mouser" "0805W8F4701T5E"
+		(property "Mouser" "0805W8F1001T5E"
 			(at 173.99 63.5 0)
 			(hide yes)
@@
 			)
 		)
-		(property "Value" "1k"
+		(property "Value" "1K"
 			(at 186.69 67.31 90)
 			(show_name no)
