File: design/CPLD.kicad_sch (KiCad schematic)
At the start: 28 parts, among them J2 Conn_02x05_Odd_Even, U2 ATF1508ASx-xxJx84, Y3 SG-5032CAN 3.6864MHz

Commit message: Fix all R/C part numbers: switch to JLCPCB basic parts, correct footprints
- Replace all non-basic LCSC numbers with JLCPCB basic equivalents (no
  extended part setup fees): Samsung MLCCs for caps, UNI-ROYAL 0805W8F
  series for resistors
- Fix C49 footprint: 1210 → 1206 to match Samsung CL31A476MPHNNNE
- Correct previously wrong LCSC numbers (C17512→C17513, C17515→C17673,
  C135808→C96123) and missing R17 part numbers
- Update all Mouser numbers to match the LCSC manufacturer throughout
- Standardise all resistor footprints to HandSolder pad variant
- Update datasheets/INDEX.md with verified basic part table

Co-Authored-By: Claude Sonnet 4.6 <noreply@anthropic.com>
Parts:
- C14, C15, C16, C17, C18, C19, C20, C21, C22: LCSC C1711 -> C49678; Mouser CL21B104KBCNNNC -> 603-CC0805KRX7R9BB104
- R10, R18, R24, R25, R26, R27, R28, R29, R30, R9: LCSC C17515 -> C17673; Mouser ERJ-6ENF4701V -> 0805W8F4701T5E
- R22, R23: LCSC C17512 -> C17513; Mouser ERJ-6ENF1001V -> 0805W8F1001T5E
- R31: LCSC C17512 -> C17379; Mouser CRCW08051K20FKEA -> 0805W8F1201T5E
Changed lines of the file:
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@@
 			)
 		)
-		(property "LCSC" "C17512"
+		(property "LCSC" "C17379"
 			(at 173.99 68.58 0)
 			(hide yes)
@@
 			)
 		)
-		(property "Mouser" "CRCW08051K20FKEA"
+		(property "Mouser" "0805W8F1201T5E"
 			(at 173.99 68.58 0)
 			(hide yes)
@@
 			)
 		)
-		(property "Mouser" "CL21B104KBCNNNC"
+		(property "Mouser" "603-CC0805KRX7R9BB104"
 			(at 21.59 26.67 0)
 			(hide yes)
@@
 			)
 		)
-		(property "LCSC" "C1711"
+		(property "LCSC" "C49678"
 			(at 21.59 26.67 0)
 			(hide yes)
@@
 			)
 		)
-		(property "LCSC" "C17515"
+		(property "LCSC" "C17673"
 			(at 214.63 93.98 0)
 			(hide yes)
@@
 			)
 		)
-		(property "Mouser" "ERJ-6ENF4701V"
+		(property "Mouser" "0805W8F4701T5E"
 			(at 214.63 93.98 0)
 			(hide yes)
@@
 			)
 		)
-		(property "LCSC" "C17515"
+		(property "LCSC" "C17673"
 			(at 234.95 93.98 0)
 			(hide yes)
@@
 			)
 		)
-		(property "Mouser" "ERJ-6ENF4701V"
+		(property "Mouser" "0805W8F4701T5E"
 			(at 234.95 93.98 0)
 			(hide yes)
@@
 			)
 		)
-		(property "LCSC" "C17515"
+		(property "LCSC" "C17673"
 			(at 204.47 121.92 0)
 			(hide yes)
@@
 			)
 		)
-		(property "Mouser" "ERJ-6ENF4701V"
+		(property "Mouser" "0805W8F4701T5E"
 			(at 204.47 121.92 0)
 			(hide yes)
@@
 			)
 		)
-		(property "LCSC" "C17515"
+		(property "LCSC" "C17673"
 			(at 214.63 68.58 0)
 			(hide yes)
@@
 			)
 		)
-		(property "Mouser" "ERJ-6ENF4701V"
+		(property "Mouser" "0805W8F4701T5E"
 			(at 214.63 68.58 0)
 			(hide yes)
@@
 			)
 		)
-		(property "Mouser" "CL21B104KBCNNNC"
+		(property "Mouser" "603-CC0805KRX7R9BB104"
 			(at 63.5 26.67 0)
 			(hide yes)
@@
 			)
 		)
-		(property "LCSC" "C1711"
+		(property "LCSC" "C49678"
 			(at 63.5 26.67 0)
 			(hide yes)
@@
 			)
 		)
-		(property "Mouser" "CL21B104KBCNNNC"
+		(property "Mouser" "603-CC0805KRX7R9BB104"
 			(at 134.62 26.67 0)
 			(hide yes)
@@
 			)
 		)
-		(property "LCSC" "C1711"
+		(property "LCSC" "C49678"
 			(at 134.62 26.67 0)
 			(hide yes)
@@
 			)
 		)
-		(property "LCSC" "C17512"
+		(property "LCSC" "C17513"
 			(at 41.91 83.82 0)
 			(hide yes)
@@
 			)
 		)
-		(property "Mouser" "ERJ-6ENF1001V"
+		(property "Mouser" "0805W8F1001T5E"
 			(at 41.91 83.82 0)
 			(hide yes)
@@
 			)
 		)
-		(property "Mouser" "CL21B104KBCNNNC"
+		(property "Mouser" "603-CC0805KRX7R9BB104"
 			(at 77.47 26.67 0)
 			(hide yes)
@@
 			)
 		)
-		(property "LCSC" "C1711"
+		(property "LCSC" "C49678"
 			(at 77.47 26.67 0)
 			(hide yes)
@@
 			)
 		)
-		(property "LCSC" "C17515"
+		(property "LCSC" "C17673"
 			(at 224.79 68.58 0)
 			(hide yes)
@@
 			)
 		)
-		(property "Mouser" "ERJ-6ENF4701V"
+		(property "Mouser" "0805W8F4701T5E"
 			(at 224.79 68.58 0)
 			(hide yes)
@@
 			)
 		)
-		(property "LCSC" "C17515"
+		(property "LCSC" "C17673"
 			(at 204.47 93.98 0)
 			(hide yes)
@@
 			)
 		)
-		(property "Mouser" "ERJ-6ENF4701V"
+		(property "Mouser" "0805W8F4701T5E"
 			(at 204.47 93.98 0)
 			(hide yes)
@@
 			)
 		)
-		(property "LCSC" "C17515"
+		(property "LCSC" "C17673"
 			(at 214.63 121.92 0)
 			(hide yes)
@@
 			)
 		)
-		(property "Mouser" "ERJ-6ENF4701V"
+		(property "Mouser" "0805W8F4701T5E"
 			(at 214.63 121.92 0)
 			(hide yes)
@@
 			)
 		)
-		(property "Mouser" "CL21B104KBCNNNC"
+		(property "Mouser" "603-CC0805KRX7R9BB104"
 			(at 119.38 26.67 0)
 			(hide yes)
@@
 			)
 		)
-		(property "LCSC" "C1711"
+		(property "LCSC" "C49678"
 			(at 119.38 26.67 0)
 			(hide yes)
@@
 			)
 		)
-		(property "Mouser" "CL21B104KBCNNNC"
+		(property "Mouser" "603-CC0805KRX7R9BB104"
 			(at 91.44 26.67 0)
 			(hide yes)
@@
 			)
 		)
-		(property "LCSC" "C1711"
+		(property "LCSC" "C49678"
 			(at 91.44 26.67 0)
 			(hide yes)
@@
 			)
 		)
-		(property "Mouser" "CL21B104KBCNNNC"
+		(property "Mouser" "603-CC0805KRX7R9BB104"
 			(at 105.41 26.67 0)
 			(hide yes)
@@
 			)
 		)
-		(property "LCSC" "C1711"
+		(property "LCSC" "C49678"
 			(at 105.41 26.67 0)
 			(hide yes)
@@
 			)
 		)
-		(property "LCSC" "C17512"
+		(property "LCSC" "C17513"
 			(at 30.48 83.82 0)
 			(hide yes)
@@
 			)
 		)
-		(property "Mouser" "ERJ-6ENF1001V"
+		(property "Mouser" "0805W8F1001T5E"
 			(at 30.48 83.82 0)
 			(hide yes)
@@
 			)
 		)
-		(property "Mouser" "CL21B104KBCNNNC"
+		(property "Mouser" "603-CC0805KRX7R9BB104"
 			(at 49.53 26.67 0)
 			(hide yes)
@@
 			)
 		)
-		(property "LCSC" "C1711"
+		(property "LCSC" "C49678"
 			(at 49.53 26.67 0)
 			(hide yes)
@@
 			)
 		)
-		(property "LCSC" "C17515"
+		(property "LCSC" "C17673"
 			(at 234.95 68.58 0)
 			(hide yes)
@@
 			)
 		)
-		(property "Mouser" "ERJ-6ENF4701V"
+		(property "Mouser" "0805W8F4701T5E"
 			(at 234.95 68.58 0)
 			(hide yes)
@@
 			)
 		)
-		(property "LCSC" "C17515"
+		(property "LCSC" "C17673"
 			(at 204.47 68.58 0)
 			(hide yes)
@@
 			)
 		)
-		(property "Mouser" "ERJ-6ENF4701V"
+		(property "Mouser" "0805W8F4701T5E"
 			(at 204.47 68.58 0)
 			(hide yes)
@@
 			)
 		)
-		(property "LCSC" "C17515"
+		(property "LCSC" "C17673"
 			(at 224.79 93.98 0)
 			(hide yes)
@@
 			)
 		)
-		(property "Mouser" "ERJ-6ENF4701V"
+		(property "Mouser" "0805W8F4701T5E"
 			(at 224.79 93.98 0)
 			(hide yes)
@@
 			)
 		)
-		(property "Mouser" "CL21B104KBCNNNC"
+		(property "Mouser" "603-CC0805KRX7R9BB104"
 			(at 35.56 26.67 0)
 			(hide yes)
@@
 			)
 		)
-		(property "LCSC" "C1711"
+		(property "LCSC" "C49678"
 			(at 35.56 26.67 0)
 			(hide yes)

Commit message: Update KiCad design files and add fabrication outputs
Schematic and PCB updates including component renumbering (ICs, passives,
LEDs, oscillators). Add JLCPCB fabrication toolkit settings and v1
production outputs (gerbers zip, IPC netlist).

Co-Authored-By: Claude Sonnet 4.6 <noreply@anthropic.com>
Parts:
- renumbered C15 to C10, C16 to C11, C17 to C12, C18 to C13, C19 to C14, C20 to C15, C21 to C16, C22 to C17, C14 to C9, LED1 to LED3, LED2 to LED4, R28 to R10, R18 to R11, R24 to R12, R26 to R13, R29 to R14, R30 to R15, R23 to R3, R22 to R4, R31 to R5, R27 to R6, R9 to R7, R10 to R8, R25 to R9, Y3 to Y2
Changed lines of the file:
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@@
 		(dnp no)
 		(fields_autoplaced yes)
-		(property "Reference" "R31"
+		(property "Reference" "R5"
 			(at 176.53 67.3099 0)
 			(show_name no)
@@
 			(project "Simple010"
 				(path "/4f37455c-e998-4ed3-8493-a94956af64c1/a4e289c4-0732-4c7f-a473-76d795f8e173"
-					(reference "R31")
+					(reference "R5")
 					(unit 1)
 				)
@@
 		(dnp no)
 		(fields_autoplaced yes)
-		(property "Reference" "C14"
+		(property "Reference" "C9"
 			(at 25.4 25.3999 0)
 			(show_name no)
@@
 			(project "Simple010"
 				(path "/4f37455c-e998-4ed3-8493-a94956af64c1/a4e289c4-0732-4c7f-a473-76d795f8e173"
-					(reference "C14")
+					(reference "C9")
 					(unit 1)
 				)
@@
 		(dnp no)
 		(fields_autoplaced yes)
-		(property "Reference" "Y3"
+		(property "Reference" "Y2"
 			(at 49.53 138.3598 0)
 			(show_name no)
@@
 			(project "Simple010"
 				(path "/4f37455c-e998-4ed3-8493-a94956af64c1/a4e289c4-0732-4c7f-a473-76d795f8e173"
-					(reference "Y3")
+					(reference "Y2")
 					(unit 1)
 				)
@@
 		(dnp no)
 		(fields_autoplaced yes)
-		(property "Reference" "R18"
+		(property "Reference" "R11"
 			(at 217.17 92.7099 0)
 			(show_name no)
@@
 			(project "Simple010"
 				(path "/4f37455c-e998-4ed3-8493-a94956af64c1/a4e289c4-0732-4c7f-a473-76d795f8e173"
-					(reference "R18")
+					(reference "R11")
 					(unit 1)
 				)
@@
 		(dnp no)
 		(fields_autoplaced yes)
-		(property "Reference" "R26"
+		(property "Reference" "R13"
 			(at 237.49 92.7099 0)
 			(show_name no)
@@
 			(project "Simple010"
 				(path "/4f37455c-e998-4ed3-8493-a94956af64c1/a4e289c4-0732-4c7f-a473-76d795f8e173"
-					(reference "R26")
+					(reference "R13")
 					(unit 1)
 				)
@@
 		(dnp no)
 		(fields_autoplaced yes)
-		(property "Reference" "R29"
+		(property "Reference" "R14"
 			(at 207.01 120.6499 0)
 			(show_name no)
@@
 			(project "Simple010"
 				(path "/4f37455c-e998-4ed3-8493-a94956af64c1/a4e289c4-0732-4c7f-a473-76d795f8e173"
-					(reference "R29")
+					(reference "R14")
 					(unit 1)
 				)
@@
 		(dnp no)
 		(fields_autoplaced yes)
-		(property "Reference" "R9"
+		(property "Reference" "R7"
 			(at 217.17 67.3099 0)
 			(show_name no)
@@
 			(project "Simple010"
 				(path "/4f37455c-e998-4ed3-8493-a94956af64c1/a4e289c4-0732-4c7f-a473-76d795f8e173"
-					(reference "R9")
+					(reference "R7")
 					(unit 1)
 				)
@@
 		(dnp no)
 		(fields_autoplaced yes)
-		(property "Reference" "C17"
+		(property "Reference" "C12"
 			(at 67.31 25.3999 0)
 			(show_name no)
@@
 			(project "Simple010"
 				(path "/4f37455c-e998-4ed3-8493-a94956af64c1/a4e289c4-0732-4c7f-a473-76d795f8e173"
-					(reference "C17")
+					(reference "C12")
 					(unit 1)
 				)
@@
 		(in_pos_files yes)
 		(dnp no)
-		(property "Reference" "LED2"
+		(property "Reference" "LED4"
 			(at 44.45 91.44 0)
 			(show_name no)
@@
 			(project "Simple010"
 				(path "/4f37455c-e998-4ed3-8493-a94956af64c1/a4e289c4-0732-4c7f-a473-76d795f8e173"
-					(reference "LED2")
+					(reference "LED4")
 					(unit 1)
 				)
@@
 		(dnp no)
 		(fields_autoplaced yes)
-		(property "Reference" "C22"
+		(property "Reference" "C17"
 			(at 138.43 25.3999 0)
 			(show_name no)
@@
 			(project "Simple010"
 				(path "/4f37455c-e998-4ed3-8493-a94956af64c1/a4e289c4-0732-4c7f-a473-76d795f8e173"
-					(reference "C22")
+					(reference "C17")
 					(unit 1)
 				)
@@
 		(dnp no)
 		(fields_autoplaced yes)
-		(property "Reference" "R22"
+		(property "Reference" "R4"
 			(at 44.45 82.5499 0)
 			(show_name no)
@@
 			(project "Simple010"
 				(path "/4f37455c-e998-4ed3-8493-a94956af64c1/a4e289c4-0732-4c7f-a473-76d795f8e173"
-					(reference "R22")
+					(reference "R4")
 					(unit 1)
 				)
@@
 		(dnp no)
 		(fields_autoplaced yes)
-		(property "Reference" "C18"
+		(property "Reference" "C13"
 			(at 81.28 25.3999 0)
 			(show_name no)
@@
 			(project "Simple010"
 				(path "/4f37455c-e998-4ed3-8493-a94956af64c1/a4e289c4-0732-4c7f-a473-76d795f8e173"
-					(reference "C18")
+					(reference "C13")
 					(unit 1)
 				)
@@
 		(dnp no)
 		(fields_autoplaced yes)
-		(property "Reference" "R10"
+		(property "Reference" "R8"
 			(at 227.33 67.3099 0)
 			(show_name no)
@@
 			(project "Simple010"
 				(path "/4f37455c-e998-4ed3-8493-a94956af64c1/a4e289c4-0732-4c7f-a473-76d795f8e173"
-					(reference "R10")
+					(reference "R8")
 					(unit 1)
 				)
@@
 		(dnp no)
 		(fields_autoplaced yes)
-		(property "Reference" "R28"
+		(property "Reference" "R10"
 			(at 207.01 92.7099 0)
 			(show_name no)
@@
 			(project "Simple010"
 				(path "/4f37455c-e998-4ed3-8493-a94956af64c1/a4e289c4-0732-4c7f-a473-76d795f8e173"
-					(reference "R28")
+					(reference "R10")
 					(unit 1)
 				)
@@
 		(in_pos_files yes)
 		(dnp no)
-		(property "Reference" "LED1"
+		(property "Reference" "LED3"
 			(at 33.02 91.44 0)
 			(show_name no)
@@
 			(project "Simple010"
 				(path "/4f37455c-e998-4ed3-8493-a94956af64c1/a4e289c4-0732-4c7f-a473-76d795f8e173"
-					(reference "LED1")
+					(reference "LED3")
 					(unit 1)
 				)
@@
 		(dnp no)
 		(fields_autoplaced yes)
-		(property "Reference" "R30"
+		(property "Reference" "R15"
 			(at 217.17 120.6499 0)
 			(show_name no)
@@
 			(project "Simple010"
 				(path "/4f37455c-e998-4ed3-8493-a94956af64c1/a4e289c4-0732-4c7f-a473-76d795f8e173"
-					(reference "R30")
+					(reference "R15")
 					(unit 1)
 				)
@@
 		(dnp no)
 		(fields_autoplaced yes)
-		(property "Reference" "C21"
+		(property "Reference" "C16"
 			(at 123.19 25.3999 0)
 			(show_name no)
@@
 			(project "Simple010"
 				(path "/4f37455c-e998-4ed3-8493-a94956af64c1/a4e289c4-0732-4c7f-a473-76d795f8e173"
-					(reference "C21")
+					(reference "C16")
 					(unit 1)
 				)
@@
 		(dnp no)
 		(fields_autoplaced yes)
-		(property "Reference" "C19"
+		(property "Reference" "C14"
 			(at 95.25 25.3999 0)
 			(show_name no)
@@
 			(project "Simple010"
 				(path "/4f37455c-e998-4ed3-8493-a94956af64c1/a4e289c4-0732-4c7f-a473-76d795f8e173"
-					(reference "C19")
+					(reference "C14")
 					(unit 1)
 				)
@@
 		(dnp no)
 		(fields_autoplaced yes)
-		(property "Reference" "C20"
+		(property "Reference" "C15"
 			(at 109.22 25.3999 0)
 			(show_name no)
@@
 			(project "Simple010"
 				(path "/4f37455c-e998-4ed3-8493-a94956af64c1/a4e289c4-0732-4c7f-a473-76d795f8e173"
-					(reference "C20")
+					(reference "C15")
 					(unit 1)
 				)
@@
 		(dnp no)
 		(fields_autoplaced yes)
-		(property "Reference" "R23"
+		(property "Reference" "R3"
 			(at 33.02 82.5499 0)
 			(show_name no)
@@
 			(project "Simple010"
 				(path "/4f37455c-e998-4ed3-8493-a94956af64c1/a4e289c4-0732-4c7f-a473-76d795f8e173"
-					(reference "R23")
+					(reference "R3")
 					(unit 1)
 				)
@@
 		(dnp no)
 		(fields_autoplaced yes)
-		(property "Reference" "C16"
+		(property "Reference" "C11"
 			(at 53.34 25.3999 0)
 			(show_name no)
@@
 			(project "Simple010"
 				(path "/4f37455c-e998-4ed3-8493-a94956af64c1/a4e289c4-0732-4c7f-a473-76d795f8e173"
-					(reference "C16")
+					(reference "C11")
 					(unit 1)
 				)
@@
 		(dnp no)
 		(fields_autoplaced yes)
-		(property "Reference" "R25"
+		(property "Reference" "R9"
 			(at 237.49 67.3099 0)
 			(show_name no)
@@
 			(project "Simple010"
 				(path "/4f37455c-e998-4ed3-8493-a94956af64c1/a4e289c4-0732-4c7f-a473-76d795f8e173"
-					(reference "R25")
+					(reference "R9")
 					(unit 1)
 				)
@@
 		(dnp no)
 		(fields_autoplaced yes)
-		(property "Reference" "R27"
+		(property "Reference" "R6"
 			(at 207.01 67.3099 0)
 			(show_name no)
@@
 			(project "Simple010"
 				(path "/4f37455c-e998-4ed3-8493-a94956af64c1/a4e289c4-0732-4c7f-a473-76d795f8e173"
-					(reference "R27")
+					(reference "R6")
 					(unit 1)
 				)
@@
 		(dnp no)
 		(fields_autoplaced yes)
-		(property "Reference" "R24"
+		(property "Reference" "R12"
 			(at 227.33 92.7099 0)
 			(show_name no)
@@
 			(project "Simple010"
 				(path "/4f37455c-e998-4ed3-8493-a94956af64c1/a4e289c4-0732-4c7f-a473-76d795f8e173"
-					(reference "R24")
+					(reference "R12")
 					(unit 1)
 				)
@@
 		(dnp no)
 		(fields_autoplaced yes)
-		(property "Reference" "C15"
+		(property "Reference" "C10"
 			(at 39.37 25.3999 0)
 			(show_name no)
@@
 			(project "Simple010"
 				(path "/4f37455c-e998-4ed3-8493-a94956af64c1/a4e289c4-0732-4c7f-a473-76d795f8e173"
-					(reference "C15")
+					(reference "C10")
 					(unit 1)
 				)
