File: design/Simple010.kicad_pcb (KiCad board)
At the start: 4 copper layers, 100 x 100 mm, 75 parts, among them J1 SPI CS2, J2 Conn_02x05_Odd_Even, J3 USB_C_Receptacle_USB2.0_16P, J4 Backup serial, J7 Conn_02x32_Odd_Even, J8 SD Card, SW1 Reset, U1 MC68010P, U2 ATF1508ASx-xxJx84, U3 SST39SF040, U4 SST39SF040, U5 AS6C4008-55PCN, U6 AS6C4008-55PCN, U7 USBLC6-2SC6, U8 MCP2221A, U9 LM809M3-4.63/NOPB, Y1 SG-5032CAN 10MHz, Y2 SG-5032CAN 3.6864MHz

Commit message: Add board render image and 3D models for PLCC84, PLCC32, oscillators, USB-C
Co-Authored-By: Claude Sonnet 4.6 <noreply@anthropic.com>
Parts:
- J1: value SPI CS2 -> CS2
Changed lines of the file:
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@@
 		)
 		(embedded_fonts no)
-		(model "${KICAD10_3DMODEL_DIR}/Package_LCC.3dshapes/PLCC-32_THT-Socket.step"
+		(model "${KIPRJMOD}/3DModels/8432-11b1-01.stp"
 			(offset
-				(xyz 0 0 0)
+				(xyz 15.5 8.5 0)
 			)
 			(scale
@@
 			)
 			(rotate
-				(xyz 0 0 0)
+				(xyz 180 180 -0)
+			)
+		)
+		(model "${KIPRJMOD}/plcc32_p1-27_l14-05_w11-51.stp"
+			(offset
+				(xyz -1 -5 0)
+			)
+			(scale
+				(xyz 1 1 1)
+			)
+			(rotate
+				(xyz -90 -0 -0)
+			)
+		)
+		(model "${KIPRJMOD}/3DModels/PLCC32_NH_SST_MCH.step"
+			(offset
+				(xyz -1 -5.5 4.5)
+			)
+			(scale
+				(xyz 1 1 1)
+			)
+			(rotate
+				(xyz -0 -0 -0)
 			)
 		)
@@
 			)
 		)
+		(model "${KICAD10_3DMODEL_DIR}/Oscillator.3dshapes/Oscillator_SMD_Fox_FT5H_5.0x3.2mm.step"
+			(offset
+				(xyz 0 0 0)
+			)
+			(scale
+				(xyz 1 1 1)
+			)
+			(rotate
+				(xyz 0 0 0)
+			)
+		)
 	)
 	(footprint "Connector_PinHeader_2.54mm:PinHeader_1x02_P2.54mm_Vertical"
@@
 		)
 		(embedded_fonts no)
-		(model "${KICAD10_3DMODEL_DIR}/Package_LCC.3dshapes/PLCC-32_THT-Socket.step"
+		(model "${KIPRJMOD}/3DModels/8432-11b1-01.stp"
 			(offset
-				(xyz 0 0 0)
+				(xyz 15 9 0)
 			)
 			(scale
@@
 			)
 			(rotate
-				(xyz 0 0 0)
+				(xyz 180 180 -0)
+			)
+		)
+		(model "${KIPRJMOD}/3DModels/PLCC32_NH_SST_MCH.step"
+			(offset
+				(xyz -2 -5 5)
+			)
+			(scale
+				(xyz 1 1 1)
+			)
+			(rotate
+				(xyz -0 -0 -0)
 			)
 		)
@@
 		(embedded_fonts no)
 		(model "${KICAD10_3DMODEL_DIR}/Package_LCC.3dshapes/PLCC-84_THT-Socket.step"
+			(hide yes)
 			(offset
 				(xyz 0 0 0)
@@
 			)
 		)
+		(model "${KIPRJMOD}/3DModels/8484-11b1-01.stp"
+			(offset
+				(xyz 18 1.5 0)
+			)
+			(scale
+				(xyz 1 1 1)
+			)
+			(rotate
+				(xyz 180 180 -0)
+			)
+		)
+		(model "${KIPRJMOD}/3DModels/PLCC84_MCH.step"
+			(offset
+				(xyz 0 -14.5 3.5)
+			)
+			(scale
+				(xyz 1 1 1)
+			)
+			(rotate
+				(xyz -0 -0 -0)
+			)
+		)
 	)
 	(footprint "Capacitor_SMD:C_0805_2012Metric_Pad1.18x1.45mm_HandSolder"
@@
 			)
 		)
-		(property "Value" "SPI CS2"
+		(property "Value" "CS2"
 			(at -2.5 0 90)
 			(layer "F.SilkS")
@@
 			)
 		)
+		(model "${KICAD10_3DMODEL_DIR}/Oscillator.3dshapes/Oscillator_SMD_Fox_FT5H_5.0x3.2mm.step"
+			(offset
+				(xyz 0 0 0)
+			)
+			(scale
+				(xyz 1 1 1)
+			)
+			(rotate
+				(xyz 0 0 0)
+			)
+		)
 	)
 	(footprint "Capacitor_SMD:C_0805_2012Metric_Pad1.18x1.45mm_HandSolder"
@@
 			)
 		)
+		(model "${KICAD10_3DMODEL_DIR}/Connector_USB.3dshapes/USB_C_Receptacle_GCT_USB4105-xx-A_16P_TopMnt_Horizontal.step"
+			(offset
+				(xyz 0 0 0)
+			)
+			(scale
+				(xyz 1 1 1)
+			)
+			(rotate
+				(xyz 0 0 0)
+			)
+		)
 	)
 	(gr_line
@@
 	)
 	(segment
+		(start 118 148)
+		(end 118 150.975)
+		(width 0.2)
+		(layer "F.Cu")
+		(net "Net-(LED1-A)")
+	)
+	(segment
+		(start 121.5 140.4625)
+		(end 121.5 140.462)
+		(width 0.2)
+		(layer "F.Cu")
+		(net "Net-(C19-Pad2)")
+	)
+	(segment
+		(start 121.5 137.5)
+		(end 121.5 140.462)
+		(width 0.2)
+		(layer "F.Cu")
+		(net "Net-(C19-Pad2)")
+	)
+	(segment
 		(start 129.3175 153.8425)
 		(end 128.5 153.025)
@@
 	)
 	(segment
-		(start 121.5 148)
-		(end 121.5 150.975)
+		(start 128.5 148)
+		(end 128.5 150.975)
 		(width 0.2)
 		(layer "F.Cu")
-		(net "Net-(LED2-A)")
+		(net "Net-(LED4-A)")
 	)
 	(segment
@@
 	)
 	(segment
+		(start 121.5 148)
+		(end 121.5 150.975)
+		(width 0.2)
+		(layer "F.Cu")
+		(net "Net-(LED2-A)")
+	)
+	(segment
 		(start 125.569 104.219)
 		(end 131.759 110.409)
@@
 	)
 	(segment
-		(start 118 148)
-		(end 118 150.975)
+		(start 125 148)
+		(end 125 150.975)
 		(width 0.2)
 		(layer "F.Cu")
-		(net "Net-(LED1-A)")
+		(net "Net-(LED3-A)")
 	)
 	(segment
@@
 	)
 	(segment
+		(start 146.864 134)
+		(end 146.8644 134)
+		(width 0.2)
+		(layer "F.Cu")
+		(net "Net-(U8-VUSB)")
+	)
+	(segment
+		(start 148.1 128.211)
+		(end 148.02 128.131)
+		(width 0.2)
+		(layer "F.Cu")
+		(net "Net-(U8-VUSB)")
+	)
+	(segment
+		(start 148.02 128.131)
+		(end 147.678 127.789)
+		(width 0.2)
+		(layer "F.Cu")
+		(net "Net-(U8-VUSB)")
+	)
+	(segment
+		(start 148.0801 128.191)
+		(end 147.6784 127.7885)
+		(width 0.2)
+		(layer "F.Cu")
+		(net "Net-(U8-VUSB)")
+	)
+	(segment
+		(start 146.8644 134)
+		(end 147.839 134)
+		(width 0.2)
+		(layer "F.Cu")
+		(net "Net-(U8-VUSB)")
+	)
+	(segment
+		(start 147.6784 127.7885)
+		(end 147.678 127.788)
+		(width 0.2)
+		(layer "F.Cu")
+		(net "Net-(U8-VUSB)")
+	)
+	(segment
+		(start 148.0201 128.131)
+		(end 148.0801 128.191)
+		(width 0.2)
+		(layer "F.Cu")
+		(net "Net-(U8-VUSB)")
+	)
+	(segment
+		(start 148.139 128.25)
+		(end 148.0801 128.191)
+		(width 0.2)
+		(layer "F.Cu")
+		(net "Net-(U8-VUSB)")
+	)
+	(segment
+		(start 148.139 133.7)
+		(end 148.139 128.25)
+		(width 0.2)
+		(layer "F.Cu")
+		(net "Net-(U8-VUSB)")
+	)
+	(segment
+		(start 147.839 134)
+		(end 148.139 133.7)
+		(width 0.2)
+		(layer "F.Cu")
+		(net "Net-(U8-VUSB)")
+	)
+	(segment
+		(start 148.02 128.131)
+		(end 148.0201 128.131)
+		(width 0.2)
+		(layer "F.Cu")
+		(net "Net-(U8-VUSB)")
+	)
+	(segment
 		(start 135.75 142)
 		(end 135.75 144.275)
@@
 		(net "Net-(J3-CC2)")
 	)
-	(segment
-		(start 146.864 134)
-		(end 146.8644 134)
-		(width 0.2)
-		(layer "F.Cu")
-		(net "Net-(U8-VUSB)")
-	)
-	(segment
-		(start 148.1 128.211)
-		(end 148.02 128.131)
-		(width 0.2)
-		(layer "F.Cu")
-		(net "Net-(U8-VUSB)")
-	)
-	(segment
-		(start 148.02 128.131)
-		(end 147.678 127.789)
-		(width 0.2)
-		(layer "F.Cu")
-		(net "Net-(U8-VUSB)")
-	)
-	(segment
-		(start 148.0801 128.191)
-		(end 147.6784 127.7885)
-		(width 0.2)
-		(layer "F.Cu")
-		(net "Net-(U8-VUSB)")
-	)
-	(segment
-		(start 146.8644 134)
-		(end 147.839 134)
-		(width 0.2)
-		(layer "F.Cu")
-		(net "Net-(U8-VUSB)")
-	)
-	(segment
-		(start 147.6784 127.7885)
-		(end 147.678 127.788)
-		(width 0.2)
-		(layer "F.Cu")
-		(net "Net-(U8-VUSB)")
-	)
-	(segment
-		(start 148.0201 128.131)
-		(end 148.0801 128.191)
-		(width 0.2)
-		(layer "F.Cu")
-		(net "Net-(U8-VUSB)")
-	)
-	(segment
-		(start 148.139 128.25)
-		(end 148.0801 128.191)
-		(width 0.2)
-		(layer "F.Cu")
-		(net "Net-(U8-VUSB)")
-	)
-	(segment
-		(start 148.139 133.7)
-		(end 148.139 128.25)
-		(width 0.2)
-		(layer "F.Cu")
-		(net "Net-(U8-VUSB)")
-	)
-	(segment
-		(start 147.839 134)
-		(end 148.139 133.7)
-		(width 0.2)
-		(layer "F.Cu")
-		(net "Net-(U8-VUSB)")
-	)
-	(segment
-		(start 148.02 128.131)
-		(end 148.0201 128.131)
-		(width 0.2)
-		(layer "F.Cu")
-		(net "Net-(U8-VUSB)")
-	)
-	(segment
-		(start 121.5 140.4625)
-		(end 121.5 140.462)
-		(width 0.2)
-		(layer "F.Cu")
-		(net "Net-(C19-Pad2)")
-	)
-	(segment
-		(start 121.5 137.5)
-		(end 121.5 140.462)
-		(width 0.2)
-		(layer "F.Cu")
-		(net "Net-(C19-Pad2)")
-	)
-	(segment
-		(start 125 148)
-		(end 125 150.975)
-		(width 0.2)
-		(layer "F.Cu")
-		(net "Net-(LED3-A)")
-	)
-	(segment
-		(start 128.5 148)
-		(end 128.5 150.975)
-		(width 0.2)
-		(layer "F.Cu")
-		(net "Net-(LED4-A)")
-	)
 	(zone
